File: OpenThermalCamera.kicad_pcb (KiCad board)
At the start: 2 copper layers, 26 x 21.6 mm, 23 parts, among them J1 Conn_01x05_Female, J2 DX07P024AJ1R1500, J3 micro5p_reversible, SW1 PB_Bootloader, U1 MLX90640, U2 TPS79333-EP, U3 STM32F042F6Px, U4 NUP2202

Commit message: Order the board.
Parts:
- removed J3: micro5p_reversible, lib_fp:micro5p_reversible_edley_technology
- removed R4: 5k1, Resistor_SMD:R_0805_2012Metric_Pad1.15x1.40mm_HandSolder
- added ID: TestPoint, TestPoint:TestPoint_Pad_D1.0mm, B.Cu at (43.4, 28.2)
- G1: footprint Symbol:OSHW-Symbol_6.7x6mm_SilkScreen -> Symbol:OSHW-Logo2_7.3x6mm_SilkScreen
- J2: value DX07P024AJ1R1500 -> UX60-MB-5ST; footprint lib_fp:DX07P024AJ1R1500 -> digikey-footprints:USB_Mini_B_Female_UX60-MB-5ST; moved to B.Cu
- moved J2 0.90 mm to (32.9, 28.3), turned to 0 degrees
Routing:
- net GND: track 82.6 -> 34.3 mm, vias 15 -> 13
- net +5V: track 61.1 -> 32.5 mm, vias 5 -> 2
- net /USB_N: track 38.4 -> 20.4 mm, vias 2 -> 0
- net Net-(J2-Pad4): track 0.00 -> 13.7 mm
- net /USB_P: track 34.7 -> 26.2 mm, vias 4 -> 2
- net Net-(J2-PadA5): track 6.05 -> 0.00 mm, vias 1 -> 0
- net (no net): vias 0 -> 1
Other:
- board size 26 x 21.6 mm -> 26 x 23.5 mm
