File: OpenThermalCamera.sch (KiCad schematic (older format))
At the start: 23 parts, among them J1 Conn_01x05_Female, J2 DX07P024AJ1R1500, J3 micro5p_reversible_edley_tech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, SW1 PB_Bootloader, U1 MLX90640, U2 TPS79333-EP, U3 STM32F042F6Px, U4 NUP2202

Commit message: Order the board.
Parts:
- removed J2: DX07P024AJ1R1500, lib_fp:DX07P024AJ1R1500, symbol DX07P024AJ1R1500:DX07P024AJ1R1500
- removed J3: micro5p_reversible_edley_technology, lib_fp:reversible_micro_usb, symbol micro5p_reversible_edley_technology:micro5p_reversible_edley_technology
- removed R4: 5k1, Resistor_SMD:R_0805_2012Metric_Pad1.15x1.40mm_HandSolder, symbol Device:R
- added J2: UX60-MB-5ST, digikey-footprints:USB_Mini_B_Female_UX60-MB-5ST, symbol dk_USB-DVI-HDMI-Connectors:UX60-MB-5ST
- added TP1: TestPoint, TestPoint:TestPoint_Pad_D1.0mm, symbol Connector:TestPoint
Connections:
- wire segments 79 -> 61
- no-connect marks 21 -> 10
Changed lines of the file:
@@
 EESchema Schematic File Version 4
 LIBS:OpenThermalCamera-cache
-EELAYER 29 0
+EELAYER 30 0
 EELAYER END
 $Descr A3 16535 11693
@@
 $EndComp
 $Comp
-L power:+5V #PWR0112
-U 1 1 5B955DC4
-P 12150 6450
-F 0 "#PWR0112" H 12150 6300 50  0001 C CNN
-F 1 "+5V" H 12165 6623 50  0000 C CNN
-F 2 "" H 12150 6450 50  0001 C CNN
-F 3 "" H 12150 6450 50  0001 C CNN
-	1    12150 6450
-	1    0    0    -1
-$EndComp
-Text Label 10800 7300 2    50   ~ 0
-USB_N
-Text Label 10800 7400 2    50   ~ 0
-USB_P
-$Comp
-L power:GND #PWR0113
-U 1 1 5B9575B1
-P 12150 7900
-F 0 "#PWR0113" H 12150 7650 50  0001 C CNN
-F 1 "GND" H 12155 7727 50  0000 C CNN
-F 2 "" H 12150 7900 50  0001 C CNN
-F 3 "" H 12150 7900 50  0001 C CNN
-	1    12150 7900
-	1    0    0    -1
-$EndComp
-$Comp
 L Power_Protection:NUP2202 U4
 U 1 1 5B9578EB
@@
 Text Label 9500 7250 0    50   ~ 0
 USB_N
-Wire Wire Line
-	11000 7300 10550 7300
-Wire Wire Line
-	11000 7400 10550 7400
-$Comp
-L Device:R R4
-U 1 1 5C02A8CD
-P 10250 7400
-F 0 "R4" H 10180 7354 50  0000 R CNN
-F 1 "5k1" H 10180 7445 50  0000 R CNN
-F 2 "Resistor_SMD:R_0805_2012Metric_Pad1.15x1.40mm_HandSolder" V 10180 7400 50  0001 C CNN
-F 3 "~" H 10250 7400 50  0001 C CNN
-F 4 "CRCW08055K10FKEAC" H 10250 7400 50  0001 C CNN "mfr#"
-	1    10250 7400
-	-1   0    0    1
-$EndComp
-Wire Wire Line
-	10250 7200 11000 7200
-$Comp
-L power:GND #PWR03
-U 1 1 5C02B867
-P 10250 7550
-F 0 "#PWR03" H 10250 7300 50  0001 C CNN
-F 1 "GND" H 10255 7377 50  0000 C CNN
-F 2 "" H 10250 7550 50  0001 C CNN
-F 3 "" H 10250 7550 50  0001 C CNN
-	1    10250 7550
-	1    0    0    -1
-$EndComp
-Wire Wire Line
-	10250 7200 10250 7250
-NoConn ~ 11000 6600
-NoConn ~ 11000 6700
-NoConn ~ 11000 6800
-NoConn ~ 11000 6900
-NoConn ~ 11000 7000
-NoConn ~ 11000 7100
-NoConn ~ 11000 7500
-NoConn ~ 11000 7600
-NoConn ~ 11000 7700
-NoConn ~ 11000 7800
-NoConn ~ 12000 6700
 NoConn ~ 6150 3300
 NoConn ~ 6150 4300
@@
 NoConn ~ 7350 3600
 NoConn ~ 7350 3500
-Wire Wire Line
-	12000 6600 12150 6600
-Wire Wire Line
-	12150 6600 12150 6450
-Wire Wire Line
-	12000 7800 12150 7800
-Wire Wire Line
-	12150 7800 12150 7900
 $Comp
 L Graphic:Logo_Open_Hardware_Small G1
@@
 L power:+5V #PWR08
 U 1 1 5D35F128
-P 14450 6600
-F 0 "#PWR08" H 14450 6450 50  0001 C CNN
-F 1 "+5V" H 14465 6773 50  0000 C CNN
-F 2 "" H 14450 6600 50  0001 C CNN
-F 3 "" H 14450 6600 50  0001 C CNN
-	1    14450 6600
-	1    0    0    -1
-$EndComp
-Wire Wire Line
-	14300 6900 14450 6900
-Wire Wire Line
-	14450 6900 14450 6600
-Wire Wire Line
-	14300 7000 14450 7000
-Wire Wire Line
-	14450 7000 14450 6900
-Connection ~ 14450 6900
+P 12400 6800
+F 0 "#PWR08" H 12400 6650 50  0001 C CNN
+F 1 "+5V" H 12415 6973 50  0000 C CNN
+F 2 "" H 12400 6800 50  0001 C CNN
+F 3 "" H 12400 6800 50  0001 C CNN
+	1    12400 6800
+	1    0    0    -1
+$EndComp
 $Comp
 L power:GND #PWR09
 U 1 1 5D362813
-P 14450 7700
-F 0 "#PWR09" H 14450 7450 50  0001 C CNN
-F 1 "GND" H 14455 7527 50  0000 C CNN
-F 2 "" H 14450 7700 50  0001 C CNN
-F 3 "" H 14450 7700 50  0001 C CNN
-	1    14450 7700
-	1    0    0    -1
-$EndComp
-Wire Wire Line
-	14300 7400 14450 7400
-Wire Wire Line
-	14450 7400 14450 7500
-Wire Wire Line
-	14300 7500 14450 7500
-Connection ~ 14450 7500
-Wire Wire Line
-	14450 7500 14450 7700
-Text Label 13000 6900 2    50   ~ 0
+P 12650 7800
+F 0 "#PWR09" H 12650 7550 50  0001 C CNN
+F 1 "GND" H 12655 7627 50  0000 C CNN
+F 2 "" H 12650 7800 50  0001 C CNN
+F 3 "" H 12650 7800 50  0001 C CNN
+	1    12650 7800
+	1    0    0    -1
+$EndComp
+Text Label 12500 7000 2    50   ~ 0
 USB_N
-Wire Wire Line
-	13250 7000 13250 6900
-Connection ~ 13250 6900
-Wire Wire Line
-	13250 6900 13000 6900
-Text Label 13000 7150 2    50   ~ 0
+Text Label 12500 7100 2    50   ~ 0
 USB_P
-Wire Wire Line
-	13250 7250 13250 7150
-Connection ~ 13250 7150
-Wire Wire Line
-	13250 7150 13000 7150
-$Comp
-L power:GND #PWR07
-U 1 1 5D36F0AB
-P 13250 7650
-F 0 "#PWR07" H 13250 7400 50  0001 C CNN
-F 1 "GND" H 13255 7477 50  0000 C CNN
-F 2 "" H 13250 7650 50  0001 C CNN
-F 3 "" H 13250 7650 50  0001 C CNN
-	1    13250 7650
-	1    0    0    -1
-$EndComp
-Wire Wire Line
-	13250 7650 13250 7500
-Connection ~ 13250 7500
-Wire Wire Line
-	13250 7500 13250 7400
-Wire Wire Line
-	13500 6900 13250 6900
-Wire Wire Line
-	13500 7000 13250 7000
-Wire Wire Line
-	13500 7150 13250 7150
-Wire Wire Line
-	13500 7250 13250 7250
-Wire Wire Line
-	13500 7500 13250 7500
-Wire Wire Line
-	13250 7400 13500 7400
-$Comp
-L micro5p_reversible_edley_technology:micro5p_reversible_edley_technology J3
-U 1 1 5D35DA56
-P 13900 6750
-F 0 "J3" H 13900 6825 50  0000 C CNN
-F 1 "micro5p_reversible_edley_technology" H 13900 6734 50  0000 C CNN
-F 2 "lib_fp:reversible_micro_usb" H 13900 6750 50  0001 C CNN
-F 3 "" H 13900 6750 50  0001 C CNN
-F 4 "1" H 13900 6750 50  0001 C CNN "DNP"
-	1    13900 6750
-	1    0    0    -1
-$EndComp
-$Comp
-L DX07P024AJ1R1500:DX07P024AJ1R1500 J2
-U 1 1 5D384E50
-P 11500 7200
-F 0 "J2" H 11500 8067 50  0000 C CNN
-F 1 "DX07P024AJ1R1500" H 11500 7976 50  0000 C CNN
-F 2 "lib_fp:DX07P024AJ1R1500" H 11500 7200 50  0001 L BNN
-F 3 "" H 11500 7200 50  0001 L BNN
-F 4 "Mouser" H 11500 7200 50  0001 L BNN "Supplier"
-F 5 "656-DX07P024AJ1R1500" H 11500 7200 50  0001 L BNN "Part Number"
-F 6 "DX07P024AJ1R1500" H 11500 7200 50  0001 L BNN "mfr#"
-F 7 "JAE Electronics" H 11500 7200 50  0001 L BNN "mfr"
-	1    11500 7200
-	1    0    0    -1
-$EndComp
 $Comp
 L power:+5V #PWR06
@@
 Wire Wire Line
 	9950 3750 9950 3950
+Wire Wire Line
+	12500 7000 12800 7000
+Wire Wire Line
+	12500 7100 12800 7100
+Wire Wire Line
+	12400 6900 12400 6800
+$Comp
+L Connector:TestPoint TP1
+U 1 1 5DB55384
+P 12150 7200
+F 0 "TP1" V 12345 7272 50  0000 C CNN
+F 1 "TestPoint" V 12254 7272 50  0000 C CNN
+F 2 "TestPoint:TestPoint_Pad_D1.0mm" H 12350 7200 50  0001 C CNN
+F 3 "~" H 12350 7200 50  0001 C CNN
+	1    12150 7200
+	0    -1   -1   0
+$EndComp
+Wire Wire Line
+	12150 7200 12800 7200
+$Comp
+L dk_USB-DVI-HDMI-Connectors:UX60-MB-5ST J2
+U 1 1 5DB3D2E8
+P 13100 7100
+F 0 "J2" H 12807 7128 60  0000 R CNN
+F 1 "UX60-MB-5ST" H 12807 7022 60  0000 R CNN
+F 2 "digikey-footprints:USB_Mini_B_Female_UX60-MB-5ST" H 13300 7300 60  0001 L CNN
+F 3 "https://media.digikey.com/pdf/Data%20Sheets/Hirose%20PDFs/UX%20Series.pdf" H 13300 7400 60  0001 L CNN
+F 4 "H2959CT-ND" H 13300 7500 60  0001 L CNN "Digi-Key_PN"
+F 5 "UX60-MB-5ST" H 13300 7600 60  0001 L CNN "MPN"
+F 6 "Connectors, Interconnects" H 13300 7700 60  0001 L CNN "Category"
+F 7 "USB, DVI, HDMI Connectors" H 13300 7800 60  0001 L CNN "Family"
+F 8 "https://media.digikey.com/pdf/Data%20Sheets/Hirose%20PDFs/UX%20Series.pdf" H 13300 7900 60  0001 L CNN "DK_Datasheet_Link"
+F 9 "/product-detail/en/hirose-electric-co-ltd/UX60-MB-5ST/H2959CT-ND/597538" H 13300 8000 60  0001 L CNN "DK_Detail_Page"
+F 10 "CONN RCPT USB2.0 MINI B SMD R/A" H 13300 8100 60  0001 L CNN "Description"
+F 11 "Hirose Electric Co Ltd" H 13300 8200 60  0001 L CNN "Manufacturer"
+F 12 "Active" H 13300 8300 60  0001 L CNN "Status"
+	1    13100 7100
+	-1   0    0    -1
+$EndComp
+Wire Wire Line
+	12400 6900 12800 6900
+Wire Wire Line
+	12800 7300 12650 7300
+Wire Wire Line
+	12650 7300 12650 7700
+Wire Wire Line
+	13300 7600 13300 7700
+Wire Wire Line
+	13300 7700 12650 7700
+Connection ~ 12650 7700
+Wire Wire Line
+	12650 7700 12650 7800
 $EndSCHEMATC
